File: pcb/puya_tamagotchi.kicad_sch (KiCad schematic)
At the start: 49 parts, among them J1 SWD pins, J2 ADDITIONAL, J3 BATTERY, J4 USB_C_Receptacle_PowerOnly_6P, Q1 AO3400A, Q2 AO3400A, Q3 AO3400A, Q4 AO3401A, SW1 TS-1187A-B-A-B, SW2 TS-1187A-B-A-B, SW3 TS-1187A-B-A-B, SW4 TS-1187A-B-A-B, U1 PY32F002BF15U6TR, U2 OLED_SH1107_128X128, U3 TP4056, U4 DW01A

Commit message: Add mounting holes
Parts:
- added H1, H2, H3, H4, H5, H6, H7, H8: MountingHole, MountingHole:MountingHole_2.2mm_M2, symbol Mechanical:MountingHole

Commit message: Add OLED decoupling, SWD resistors
Parts:
- added C7: 100nF, PCM_JLCPCB:C_0402, symbol PCM_JLCPCB-Capacitors:0402,100nF
- added R16, R17: 10kΩ, PCM_JLCPCB:R_0402, symbol PCM_JLCPCB-Resistors:0402,10kΩ
- added TP7: TestPoint, TestPoint:TestPoint_Pad_D1.0mm, symbol Connector:TestPoint
Connections:
- net GND: now also C7.1, R17.2
- net LDR_OUT: now also TP7.1
- net SWCLK: now also R17.1
- net SWDIO: now also R16.2
- net VCC: now also C7.2, R16.1
Other:
- moved on the sheet: J1
